File: Arduino_MEGA2560_ref.brd (EAGLE design)
At the start: 101.6 x 53.3 mm, 72 parts, among them IC1 MC33269ST-5.0T3, IC2 MC33269D-5.0, IC3 ATMEGA2560-16AU, IC4 ATMEGA8U2-MU, IC5 LM358D, IC6 LP2985-33DBVR, Q1 16MHz, Q2 16MHz, T2 FDN340P, X1 DC21MMX, Y1 16MHz, Y2 16MHz

Commit message: Updated Arduino_MEGA2560_ref.brd
Parts:
- removed ON: GREEN, led:CHIP-LED0805
- added D2: HLMP6, display-hp:HLMP6
- RN1: value 10K -> 100K
- flipped L to the bottom
Connections:
- removed net PB5: IC3.24, PWMH.4
- net GND: no longer ON.C
- net N$3: no longer ON.A
Routing:
- net PB5: track 35.4 -> 0.00 mm
- net PE1: track 56.8 -> 57.9 mm
- net N$2: track 5.21 -> 5.72 mm, vias 0 -> 1
Other:
- board text added: "CADLAB.io"
- board text removed: "AREF"
